File: et55.kicad_sch (KiCad schematic)
At the start: 70 parts, among them J3 Conn_01x04, J6 Conn_01x08, M1 mini-spox, M2 mini-spox, T10 2N6426, T11 SGS110, T12 SGS115, T2 TIP110, T3 TIP125, T4 2N6426, T5 2N6426, T6 2N6426, T7 BC237B, T8 BC237B, T9 TIP110, U0 HD63B01YOP, U1 SN74LS05N, U2 SN74LS05N, U3 SN74LS05N, U6 TEA3717, U7 TEA3717

Commit message: fix: connect cpu pins to keyboard matrix
Parts:
- removed C10, C11, C12: ?nF, symbol Device:C
- removed U1: SN74LS05N, symbol et55:SN74LS05N
- added BZ?: (no value), symbol Device:Buzzer
- added C14: ?nF, symbol Device:C
- added D11, D12, D13, D14, D15, D16, D17, D18, D19: ?v ?mA, symbol Device:D_Schottky
- added R18, R19, R20, R21, R24, R25, R26, R27, R28, R29, R30, R31, R32, R33, R34: ?Ω, symbol Device:R
- added R35: R, symbol Device:R
- added R4: (no value), symbol Device:R
- M1, M2: value mini-spox -> sw-or-led?
Connections:
- net P30 is gone; now on net GND: U0.58 (P30/D0)
- net GND: now also C1.2, C10.2, C5.2, T10.1 (E), T11.3 (E), T5.1 (E), T6.1 (E), T7.3 (E), BZ?.2 (+), D14.2 (A), D19.2 (A), R18.1, R20.1, R21.1, R28.1, R29.1, R34.1; no longer C1.1, C10.1, C5.1, U0.60 (P73/~{LIR})
- net VCC: now also U2.14 (VCC), R4.2
- net VCC_5V: now also C1.1, C5.1, R5.2, R6.1, RN2.1 (common), RN3.1 (common)
- net V_FUSE: now also R13.1, D16.1 (K), D18.1 (K); no longer R13.2
- net P42: now reaches U0.39 (P42/A10)
- net P42: now also R30.1
- net P41: now reaches U0.40 (P41/A9)
- net P41: now also R26.1
- net P40: now reaches U0.41 (P40/A8)
- net P40: now also C14.1
- net J5_8: now reaches D10.2 (A), T2.3 (E)
- net J5_8: now also C8.1
- net KEY_COL_3: now reaches U2.10 (5Y)
- net KEY_COL_4: now reaches U2.12 (6Y)
- net at U2.2 (1Y): now also R35.2, R4.1
- net KEY_COL_0: now reaches U2.4 (2Y)
- net KEY_COL_1: now reaches U2.6 (3Y)
- net KEY_COL_2: now reaches U2.8 (4Y)
- net at T11.1 (B): now also R31.1
- net J6_1: now reaches T11.2 (C)
- net J6_1: now also T12.2 (C), D18.2 (A), D19.1 (K)
- net at R12.1, T3.1 (B): now also R13.2; no longer R13.1
- net at T8.1 (C): now also R27.2
- net at T8.2 (B): now also D15.2 (A), R26.2
- net at T8.3 (E): now also T5.2 (B), R21.2
- net at T10.2 (B): now also D17.2 (A), R30.2
- net at T10.3 (C): now also R31.2, R32.2, R33.2
- net J5_7: now reaches T5.3 (C)
- net J5_7: now also D13.2 (A)
- net at T7.1 (C): now also T9.1 (B), D14.1 (K), R25.1
- net at T7.2 (B): now also T6.3 (C), R24.1
- net at T12.1 (B): now also R33.1
- net at T12.3 (E): now also D13.1 (K), R24.2, R25.2, R27.1, R32.1
- net at T6.2 (B): now also D12.2 (A), R19.1
- net J5_5: now reaches T9.2 (C)
- net J5_5: now also D16.2 (A)
- net at T9.3 (E): now also R28.2, R29.2, R34.2
- net KEY_COL_5: now reaches U3.2 (1Y)
- net KEY_COL_6: now reaches U3.4 (2Y)
- net KEY_COL_7: now reaches U3.6 (3Y)
- net P20 renamed ~{KEY_KB}
- net P21 renamed ~{KEY_SHIFT}
- net P22 renamed ~{KEY_PITCH_15}
- net P23 renamed ~{KEY_PITCH_10}
- net P24 renamed ~{KEY_LF_2}
- net P25 renamed ~{KEY_LF_1}
- net P26 renamed ~{BUZZER}
- net P43: no longer names the net of M1.2 (Pin_2), U0.38 (P43/A11)
- net P43: now also R5.1; no longer R5.2
- net P47: no longer names the net of M2.2 (Pin_2), R6.2, U0.34 (P47/A15)
- net P50 renamed KEY_ROW_0
- net P51 renamed KEY_ROW_1
- net P52 renamed KEY_ROW_2
- net P53 renamed KEY_ROW_3
- net P54 renamed KEY_ROW_4
- net P55 renamed KEY_ROW_5
- net P56 renamed KEY_ROW_6
- net P57 renamed KEY_ROW_7
- net P60 renamed ~{KEY_COL_0}
- net P61 renamed ~{KEY_COL_1}
- net P62 renamed ~{KEY_COL_2}
- net P63 renamed ~{KEY_COL_3}
- net P64 renamed ~{KEY_COL_4}
- net P65 renamed ~{KEY_COL_7}
- net P66 renamed ~{KEY_COL_6}
- net P67 renamed ~{KEY_COL_5}
- net V_T2_3: no longer names the net of D10.1 (K), T3.2 (C)
- net V_T2_3: now also C10.1; no longer C10.2
- new net: C14.2, D11.1 (K), R19.2, R20.2
- new net: BZ?.1 (-), R35.1
- new net: D11.2 (A), R18.2
- new net P73: U0.60 (P73/~{LIR})
- new net RST: D12.1 (K), D15.1 (K), D17.1 (K)
- no-connect marks 3 -> 5
Other:
- note added: "H Bridge CTRL"
- note added: "Pull-up input"
- note added: "Pull-up input (HIGH)"
- note added: "Pull-up input (LOW)"
- note added: "Pull-up input ON/OFF switch or open flap signal"
- note added: "T10 Base Ctrl"
- note added: "T4 Base CTRL"
- note added: "T6 Base Ctrl"
- note added: "T8 Base Ctrl"
- note added: "output"
- note added: "output LED ctrl: EDIT"
- note added: "output LED ctrl: I-ON"
- note added: "output Led ctrl: CAPS"
- note removed: "LED ctrl: EDIT"
- note removed: "LED ctrl: I-ON"
- note removed: "Led ctrl: CAPS"
- moved on the sheet: C1, C10, C2, C3, C4, C5, D1, D10, M1, M2, R10, R11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

Commit message: feat: add resistance values
Parts:
- removed 1.6kΩ, 470Ω: R, symbol Device:R
- removed C12, C13, C15, C17, C19, C20, C?: ?nF, symbol Device:C
- removed C? (x2): 100nF, symbol Device:C
- removed D1, D10: ?v ?mA, symbol Device:D_Schottky
- removed D? (x4): 60v 30mA, symbol Device:D_Schottky
- removed J6: Conn_01x08, Connector_Molex:Molex_SPOX_5267-08A_1x08_P2.50mm_Vertical, symbol Connector_Generic:Conn_01x08
- removed R13, R14, R15, R16, R17, R22, R23: ?Ω, symbol Device:R
- removed R?: 270Ω, symbol Device:R
- removed R?: 2.2kΩ, symbol Device:R
- removed U6, U7: TEA3717, symbol et55:TEA3717
- added D1, D10: D_Zener, symbol Device:D_Zener
- BZ?: value (none) -> Buzzer
- C18: renamed from C8; value ?nF -> 47uF
- D16: Comment (none) -> Feedback diode
- R10: value ?Ω -> 5.6kΩ; Tolerance (none) -> 5%
- R11: value ?Ω -> 1kΩ; Tolerance (none) -> 5%
- R12: value ?Ω -> 12kΩ; Tolerance (none) -> 5%
- R13: value ?Ω -> 1.6kΩ; Tolerance (none) -> 5%
- R18: value ?Ω -> 100Ω; Tolerance (none) -> 5%
- R19: value ?Ω -> 10kΩ; Tolerance (none) -> 5%
- R20: value ?Ω -> 21kΩ; Tolerance (none) -> 5%
- R21: value ?Ω -> 4.7kΩ; Tolerance (none) -> 5%
- R24: value ?Ω -> 100kΩ; Tolerance (none) -> 5%
- R25: value ?Ω -> 1kΩ; Tolerance (none) -> 2%
- R26, R30: value ?Ω -> 39kΩ; Tolerance (none) -> 5%
- R27: value ?Ω -> 20kΩ; Tolerance (none) -> 5%
- R28: value ?Ω -> 15Ω; Tolerance (none) -> 2%
- R29: value ?Ω -> 7.5Ω; Tolerance (none) -> 2%
- R31: value ?Ω -> 220kΩ; Tolerance (none) -> 5%
- R32: value ?Ω -> 750Ω; Tolerance (none) -> 5%
- R33: value ?Ω -> 27kΩ; Tolerance (none) -> 5%
- R34: value ?Ω -> 1Ω; Tolerance (none) -> 2%
- R35: value R -> 100Ω; Tolerance (none) -> 5%
- R4: value (none) -> 2.4kΩ; Tolerance (none) -> 5%
- R5, R6: value ?Ω -> 470Ω; Tolerance (none) -> 5%
- R8: value ?Ω -> 1.6kΩ; Power (none) -> 1W; Tolorance (none) -> 5%
- R9: value ?Ω -> 2.2kΩ; Tolerance (none) -> 5%
- T3: value TIP125 -> TIP115
- renumbered D12 to DZ12, D14 to DZ14, D15 to DZ15, D17 to DZ17, T11 to Q11
Connections:
- net J5_8 is gone; now on net J5_8 T2_Vcc_3_ref: C18.1, T2.3 (E)
- net GND: now also D1.2 (A)
- net at C10.1, T3.2 (C): now also D10.1 (K)
- net J5_8 T2_Vcc_3_ref: now reaches D13.1 (K), R24.2, R25.2, R27.1, R32.1, T12.3 (E)
- net J5_8 T2_Vcc_3_ref: now also D10.2 (A)
- net at R8.2, T2.1 (B): now also D1.1 (K)
- net V_FUSE renamed V_FUSE_24V?
- net V_FUSE_24V?: no longer D16.1 (K), D18.1 (K)
- new net J5_6: D16.1 (K), D18.1 (K)
Other:
- added sheet et55-daisy-wheel-type-driver (et55-daisy-wheel-type-driver.kicad_sch)
- note added: "Output Paper motor"
- note added: "Output Type SOLENOID - Pulse"
- note added: "Output ctrl TAPE UP/DOWN"
- note added: "Paper up motor"
- note added: "Power Boost (Enable)"
- note added: "SOLENOID (push up base)"
- note added: "Type"
- note removed: "T10 Base Ctrl"
- note removed: "T4 Base CTRL"
- note removed: "T6 Base Ctrl"
- note removed: "T8 Base Ctrl"
- moved on the sheet: D13, R10, R11, R12, R20, R9, T4
