File: et55_dc-dual-phase-h-driver.kicad_sch (KiCad schematic)
At the start: 11 parts, among them J4 Conn_01x04, U5 L293C

Commit message: feat: add resistance values
Other:
- note added: "Kontrola pozycji karetki ( prawo lewo)"
Changed lines of the file:
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@@
     (stroke (width 0) (type default) (color 0 0 0 0))
+  )
+  (text "Kontrola pozycji karetki ( prawo lewo) " (at 220.98 92.71 0)
+    (effects (font (size 1.27 1.27)) (justify left bottom))
   )
   (global_label "RST" (shape input) (at 130.81 88.9 0) (fields_autoplaced)
