File: et55_leds.kicad_sch (KiCad schematic)
At the start: 6 parts

Commit message: feat: add resistance values
Parts:
- R1, R2, R3: renamed from R?; value ??Ω -> 270Ω; Tolerance (none) -> 5%
Changed lines of the file:
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@@
   (symbol (lib_id "Device:R") (at 116.84 60.96 90) (unit 1)
     (in_bom yes) (on_board yes) (fields_autoplaced)
-    (property "Reference" "R?" (id 0) (at 116.84 54.61 90))
-    (property "Value" "??Ω" (id 1) (at 116.84 57.15 90))
+    (property "Reference" "R1" (id 0) (at 116.84 54.61 90))
+    (property "Value" "270Ω" (id 1) (at 116.84 57.15 90))
     (property "Footprint" "" (id 2) (at 116.84 62.738 90)
       (effects (font (size 1.27 1.27)) hide)
     )
     (property "Datasheet" "~" (id 3) (at 116.84 60.96 0)
+      (effects (font (size 1.27 1.27)) hide)
+    )
+    (property "Tolerance" "5%" (id 4) (at 116.84 60.96 90)
       (effects (font (size 1.27 1.27)) hide)
     )
@@
   (symbol (lib_id "Device:R") (at 116.84 71.12 90) (unit 1)
     (in_bom yes) (on_board yes) (fields_autoplaced)
-    (property "Reference" "R?" (id 0) (at 116.84 64.77 90))
-    (property "Value" "??Ω" (id 1) (at 116.84 67.31 90))
+    (property "Reference" "R2" (id 0) (at 116.84 64.77 90))
+    (property "Value" "270Ω" (id 1) (at 116.84 67.31 90))
     (property "Footprint" "" (id 2) (at 116.84 72.898 90)
       (effects (font (size 1.27 1.27)) hide)
     )
     (property "Datasheet" "~" (id 3) (at 116.84 71.12 0)
+      (effects (font (size 1.27 1.27)) hide)
+    )
+    (property "Tolerance" "5%" (id 4) (at 116.84 71.12 90)
       (effects (font (size 1.27 1.27)) hide)
     )
@@
   (symbol (lib_id "Device:R") (at 116.84 81.28 90) (unit 1)
     (in_bom yes) (on_board yes) (fields_autoplaced)
-    (property "Reference" "R?" (id 0) (at 116.84 74.93 90))
-    (property "Value" "??Ω" (id 1) (at 116.84 77.47 90))
+    (property "Reference" "R3" (id 0) (at 116.84 74.93 90))
+    (property "Value" "270Ω" (id 1) (at 116.84 77.47 90))
     (property "Footprint" "" (id 2) (at 116.84 83.058 90)
       (effects (font (size 1.27 1.27)) hide)
@@
       (effects (font (size 1.27 1.27)) hide)
     )
+    (property "Tolerance" "5%" (id 4) (at 116.84 81.28 90)
+      (effects (font (size 1.27 1.27)) hide)
+    )
