File: et55_power-5v.kicad_sch (KiCad schematic)
At the start: 5 parts, among them U4 L387A

Commit message: feat: add resistance values
Parts:
- R7: value ?Ω -> 2.7kΩ; Tolerance (none) -> 5%
Changed lines of the file:
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@@
     (in_bom yes) (on_board yes)
     (property "Reference" "R7" (id 0) (at 167.64 106.68 90))
-    (property "Value" "?Ω" (id 1) (at 167.64 104.14 90))
+    (property "Value" "2.7kΩ" (id 1) (at 167.64 104.14 90))
     (property "Footprint" "" (id 2) (at 167.64 98.552 90)
       (effects (font (size 1.27 1.27)) hide)
@@
       (effects (font (size 1.27 1.27)) hide)
     )
+    (property "Tolerance" "5%" (id 4) (at 167.64 100.33 90)
+      (effects (font (size 1.27 1.27)) hide)
+    )
